Commit message: teleop working now

File: install/wd_lift_robot/share/wd_lift_robot/urdf/robot.urdf.xacro (robot description, xacro)
@@ -1,330 +1 @@
-<?xml version="1.0"?>
-<robot name="4wd_lift_robot" xmlns:xacro="http://www.ros.org/wiki/xacro">
-  <!-- Properties for easy customization -->
-  <xacro:property name="base_width" value="0.6"/>
-  <xacro:property name="base_length" value="0.8"/>
-  <xacro:property name="base_height" value="0.15"/>
-  <xacro:property name="wheel_radius" value="0.1"/>
-  <xacro:property name="wheel_width" value="0.08"/>
-  <xacro:property name="wheel_offset_x" value="0.3"/>
-  <xacro:property name="wheel_offset_y" value="0.35"/>
-  <xacro:property name="wheel_offset_z" value="-0.05"/>
-  <xacro:property name="lift_height_min" value="0.0"/>
-  <xacro:property name="lift_height_max" value="0.5"/>
-  <xacro:property name="cradle_width" value="0.4"/>
-  <xacro:property name="cradle_length" value="0.3"/>
-  <xacro:property name="cradle_height" value="0.1"/>
-  <!-- Materials -->
-  <material name="blue">
-    <color rgba="0 0 0.8 1"/>
-  </material>
-  <material name="black">
-    <color rgba="0 0 0 1"/>
-  </material>
-  <material name="white">
-    <color rgba="1 1 1 1"/>
-  </material>
-  <material name="red">
-    <color rgba="0.8 0.0 0.0 1.0"/>
-  </material>
-  <material name="green">
-    <color rgba="0.0 0.8 0.0 1.0"/>
-  </material>
-  <!-- Base Link (Main Chassis) -->
-  <link name="base_link">
-    <visual>
-      <origin xyz="0 0 0" rpy="0 0 0"/>
-      <geometry>
-        <box size="${base_length} ${base_width} ${base_height}"/>
-      </geometry>
-      <material name="blue"/>
-    </visual>
-    <collision>
-      <origin xyz="0 0 0" rpy="0 0 0"/>
-      <geometry>
-        <box size="${base_length} ${base_width} ${base_height}"/>
-      </geometry>
-    </collision>
-    <inertial>
-      <mass value="20.0"/>
-      <origin xyz="0 0 0" rpy="0 0 0"/>
-      <inertia ixx="1.0" ixy="0.0" ixz="0.0" iyy="1.0" iyz="0.0" izz="1.0"/>
-    </inertial>
-  </link>
-  <!-- Wheel Macro -->
-  <xacro:macro name="wheel" params="name x y z">
-    <link name="${name}_wheel">
-      <visual>
-        <origin xyz="0 0 0" rpy="1.5708 0 0"/>
-        <geometry>
-          <cylinder length="${wheel_width}" radius="${wheel_radius}"/>
-        </geometry>
-        <material name="black"/>
-      </visual>
-      <collision>
-        <origin xyz="0 0 0" rpy="1.5708 0 0"/>
-        <geometry>
-          <cylinder length="${wheel_width}" radius="${wheel_radius}"/>
-        </geometry>
-      </collision>
-      <inertial>
-        <mass value="2.5"/>
-        <origin xyz="0 0 0" rpy="1.5708 0 0"/>
-        <inertia ixx="0.01" ixy="0.0" ixz="0.0" iyy="0.005" iyz="0.0" izz="0.005"/>
-      </inertial>
-    </link>
-    <joint name="${name}_wheel_joint" type="continuous">
-      <parent link="base_link"/>
-      <child link="${name}_wheel"/>
-      <origin xyz="${x} ${y} ${z}" rpy="0 0 0"/>
-      <axis xyz="0 1 0"/>
-    </joint>
-  </xacro:macro>
-  <!-- Create all four wheels -->
-  <xacro:wheel name="front_left" x="${wheel_offset_x}" y="${wheel_offset_y}" z="${wheel_offset_z}"/>
-  <xacro:wheel name="front_right" x="${wheel_offset_x}" y="${-wheel_offset_y}" z="${wheel_offset_z}"/>
-  <xacro:wheel name="rear_left" x="${-wheel_offset_x}" y="${wheel_offset_y}" z="${wheel_offset_z}"/>
-  <xacro:wheel name="rear_right" x="${-wheel_offset_x}" y="${-wheel_offset_y}" z="${wheel_offset_z}"/>
-  <!-- Hydraulic Lift Base -->
-  <link name="lift_base">
-    <visual>
-      <origin xyz="0 0 0" rpy="0 0 0"/>
-      <geometry>
-        <cylinder length="0.05" radius="0.08"/>
-      </geometry>
-      <material name="white"/>
-    </visual>
-    <collision>
-      <origin xyz="0 0 0" rpy="0 0 0"/>
-      <geometry>
-        <cylinder length="0.05" radius="0.08"/>
-      </geometry>
-    </collision>
-    <inertial>
-      <mass value="2.0"/>
-      <origin xyz="0 0 0" rpy="0 0 0"/>
-      <inertia ixx="0.01" ixy="0.0" ixz="0.0" iyy="0.01" iyz="0.0" izz="0.01"/>
-    </inertial>
-  </link>
-  <joint name="lift_base_joint" type="fixed">
-    <parent link="base_link"/>
-    <child link="lift_base"/>
-    <origin xyz="0 0 ${base_height/2 + 0.025}" rpy="0 0 0"/>
-  </joint>
-  <!-- Hydraulic Lift Piston -->
-  <link name="lift_piston">
-    <visual>
-      <origin xyz="0 0 0.1" rpy="0 0 0"/>
-      <geometry>
-        <cylinder length="0.2" radius="0.06"/>
-      </geometry>
-      <material name="red"/>
-    </visual>
-    <collision>
-      <origin xyz="0 0 0.1" rpy="0 0 0"/>
-      <geometry>
-        <cylinder length="0.2" radius="0.06"/>
-      </geometry>
-    </collision>
-    <inertial>
-      <mass value="3.0"/>
-      <origin xyz="0 0 0.1" rpy="0 0 0"/>
-      <inertia ixx="0.02" ixy="0.0" ixz="0.0" iyy="0.02" iyz="0.0" izz="0.01"/>
-    </inertial>
-  </link>
-  <joint name="lift_joint" type="prismatic">
-    <parent link="lift_base"/>
-    <child link="lift_piston"/>
-    <origin xyz="0 0 0.025" rpy="0 0 0"/>
-    <axis xyz="0 0 1"/>
-    <limit lower="${lift_height_min}" upper="${lift_height_max}" effort="1000.0" velocity="0.5"/>
-  </joint>
-  <!-- V-Cradle Platform -->
-  <link name="cradle_platform">
-    <visual>
-      <origin xyz="0 0 0" rpy="0 0 0"/>
-      <geometry>
-        <box size="${cradle_length} ${cradle_width} ${cradle_height}"/>
-      </geometry>
-      <material name="green"/>
-    </visual>
-    <collision>
-      <origin xyz="0 0 0" rpy="0 0 0"/>
-      <geometry>
-        <box size="${cradle_length} ${cradle_width} ${cradle_height}"/>
-      </geometry>
-    </collision>
-    <inertial>
-      <mass value="5.0"/>
-      <origin xyz="0 0 0" rpy="0 0 0"/>
-      <inertia ixx="0.1" ixy="0.0" ixz="0.0" iyy="0.1" iyz="0.0" izz="0.1"/>
-    </inertial>
-  </link>
-  <joint name="cradle_joint" type="fixed">
-    <parent link="lift_piston"/>
-    <child link="cradle_platform"/>
-    <origin xyz="0 0 0.25" rpy="0 0 0"/>
-  </joint>
-  <!-- LiDAR Sensor -->
-  <link name="laser">
-    <visual>
-      <origin xyz="0 0 0" rpy="0 0 0"/>
-      <geometry>
-        <cylinder length="0.04" radius="0.035"/>
-      </geometry>
-      <material name="black"/>
-    </visual>
-    <collision>
-      <origin xyz="0 0 0" rpy="0 0 0"/>
-      <geometry>
-        <cylinder length="0.04" radius="0.035"/>
-      </geometry>
-    </collision>
-    <inertial>
-      <mass value="0.3"/>
-      <origin xyz="0 0 0" rpy="0 0 0"/>
-      <inertia ixx="0.001" ixy="0.0" ixz="0.0" iyy="0.001" iyz="0.0" izz="0.001"/>
-    </inertial>
-  </link>
-  <joint name="laser_joint" type="fixed">
-    <parent link="base_link"/>
-    <child link="laser"/>
-    <origin xyz="0.15 0 ${base_height/2 + 0.02}" rpy="0 0 0"/>
-  </joint>
-  <!-- ROS2 Control interface -->
-  <ros2_control name="GazeboSystem" type="system">
-    <hardware>
-      <plugin>gazebo_ros2_control/GazeboSystem</plugin>
-    </hardware>
-    <!-- Wheel joints -->
-    <joint name="front_left_wheel_joint">
-      <command_interface name="velocity">
-        <param name="min">-10</param>
-        <param name="max">10</param>
-      </command_interface>
-      <state_interface name="velocity"/>
-      <state_interface name="position"/>
-    </joint>
-    <joint name="front_right_wheel_joint">
-      <command_interface name="velocity">
-        <param name="min">-10</param>
-        <param name="max">10</param>
-      </command_interface>
-      <state_interface name="velocity"/>
-      <state_interface name="position"/>
-    </joint>
-    <joint name="rear_left_wheel_joint">
-      <command_interface name="velocity">
-        <param name="min">-10</param>
-        <param name="max">10</param>
-      </command_interface>
-      <state_interface name="velocity"/>
-      <state_interface name="position"/>
-    </joint>
-    <joint name="rear_right_wheel_joint">
-      <command_interface name="velocity">
-        <param name="min">-10</param>
-        <param name="max">10</param>
-      </command_interface>
-      <state_interface name="velocity"/>
-      <state_interface name="position"/>
-    </joint>
-    <!-- Lift joint -->
-    <joint name="lift_joint">
-      <command_interface name="position">
-        <param name="min">0</param>
-        <param name="max">0.5</param>
-      </command_interface>
-      <state_interface name="position"/>
-      <state_interface name="velocity"/>
-    </joint>
-  </ros2_control>
-  <!-- Gazebo plugin for ros2_control -->
-  <gazebo>
-    <plugin filename="libgazebo_ros2_control.so" name="gazebo_ros2_control">
-      <parameters>$(find wd_lift_robot)/config/controllers.yaml</parameters>
-    </plugin>
-  </gazebo>
-  <!-- Gazebo-specific configurations -->
-  <gazebo reference="base_link">
-    <material>Gazebo/Blue</material>
-  </gazebo>
-  <!-- Wheel physics -->
-  <gazebo reference="front_left_wheel">
-    <material>Gazebo/Black</material>
-    <mu1>1.0</mu1>
-    <mu2>1.0</mu2>
-    <kp>500000.0</kp>
-    <kd>10.0</kd>
-    <minDepth>0.001</minDepth>
-    <maxVel>0.1</maxVel>
-    <fdir1>1 0 0</fdir1>
-  </gazebo>
-  <gazebo reference="front_right_wheel">
-    <material>Gazebo/Black</material>
-    <mu1>1.0</mu1>
-    <mu2>1.0</mu2>
-    <kp>500000.0</kp>
-    <kd>10.0</kd>
-    <minDepth>0.001</minDepth>
-    <maxVel>0.1</maxVel>
-    <fdir1>1 0 0</fdir1>
-  </gazebo>
-  <gazebo reference="rear_left_wheel">
-    <material>Gazebo/Black</material>
-    <mu1>1.0</mu1>
-    <mu2>1.0</mu2>
-    <kp>500000.0</kp>
-    <kd>10.0</kd>
-    <minDepth>0.001</minDepth>
-    <maxVel>0.1</maxVel>
-    <fdir1>1 0 0</fdir1>
-  </gazebo>
-  <gazebo reference="rear_right_wheel">
-    <material>Gazebo/Black</material>
-    <mu1>1.0</mu1>
-    <mu2>1.0</mu2>
-    <kp>500000.0</kp>
-    <kd>10.0</kd>
-    <minDepth>0.001</minDepth>
-    <maxVel>0.1</maxVel>
-    <fdir1>1 0 0</fdir1>
-  </gazebo>
-  <!-- LiDAR sensor plugin -->
-  <gazebo reference="laser">
-    <material>Gazebo/Black</material>
-    <sensor type="ray" name="rplidar_a1">
-      <pose>0 0 0 0 0 0</pose>
-      <visualize>true</visualize>
-      <update_rate>15</update_rate>
-      <ray>
-        <scan>
-          <horizontal>
-            <samples>360</samples>
-            <resolution>1</resolution>
-            <min_angle>-3.14159265</min_angle>
-            <max_angle>3.14159265</max_angle>
-          </horizontal>
-        </scan>
-        <range>
-          <min>0.15</min>
-          <max>12.0</max>
-          <resolution>0.01</resolution>
-        </range>
-        <noise>
-          <type>gaussian</type>
-          <mean>0.0</mean>
-          <stddev>0.01</stddev>
-        </noise>
-      </ray>
-      <plugin name="gazebo_ros_laser" filename="libgazebo_ros_ray_sensor.so">
-        <ros>
-          <namespace>/</namespace>
-          <remapping>~/out:=scan</remapping>
-        </ros>
-        <output_type>sensor_msgs/LaserScan</output_type>
-        <frame_name>laser</frame_name>
-      </plugin>
-    </sensor>
-  </gazebo>
-</robot>
+/home/anish/your_robot_ws/src/wd_lift_robot/urdf/robot.urdf.xacro

File: src/wd_lift_robot/urdf/robot.urdf.xacro (robot description, xacro)
@@ -166,5 +166,5 @@
     <origin xyz="0 0 0.25" rpy="0 0 0"/>
   </joint>
-  <!-- LiDAR Sensor -->
+  <!-- LiDAR Sensor - IMPROVED RANGE -->
   <link name="laser">
     <visual>
@@ -200,6 +200,6 @@
     <joint name="front_left_wheel_joint">
       <command_interface name="velocity">
-        <param name="min">-10</param>
-        <param name="max">10</param>
+        <param name="min">-50</param>
+        <param name="max">50</param>
       </command_interface>
       <state_interface name="velocity"/>
@@ -208,6 +208,6 @@
     <joint name="front_right_wheel_joint">
       <command_interface name="velocity">
-        <param name="min">-10</param>
-        <param name="max">10</param>
+        <param name="min">-50</param>
+        <param name="max">50</param>
       </command_interface>
       <state_interface name="velocity"/>
@@ -216,6 +216,6 @@
     <joint name="rear_left_wheel_joint">
       <command_interface name="velocity">
-        <param name="min">-10</param>
-        <param name="max">10</param>
+        <param name="min">-50</param>
+        <param name="max">50</param>
       </command_interface>
       <state_interface name="velocity"/>
@@ -224,6 +224,6 @@
     <joint name="rear_right_wheel_joint">
       <command_interface name="velocity">
-        <param name="min">-10</param>
-        <param name="max">10</param>
+        <param name="min">-50</param>
+        <param name="max">50</param>
       </command_interface>
       <state_interface name="velocity"/>
@@ -291,5 +291,5 @@
     <fdir1>1 0 0</fdir1>
   </gazebo>
-  <!-- LiDAR sensor plugin -->
+  <!-- LiDAR sensor plugin - IMPROVED -->
   <gazebo reference="laser">
     <material>Gazebo/Black</material>
@@ -297,9 +297,9 @@
       <pose>0 0 0 0 0 0</pose>
       <visualize>true</visualize>
-      <update_rate>15</update_rate>
+      <update_rate>30</update_rate>
       <ray>
         <scan>
           <horizontal>
-            <samples>360</samples>
+            <samples>720</samples>
             <resolution>1</resolution>
             <min_angle>-3.14159265</min_angle>
@@ -308,6 +308,6 @@
         </scan>
         <range>
-          <min>0.15</min>
-          <max>12.0</max>
+          <min>0.1</min>
+          <max>15.0</max>
           <resolution>0.01</resolution>
         </range>
@@ -315,5 +315,5 @@
           <type>gaussian</type>
           <mean>0.0</mean>
-          <stddev>0.01</stddev>
+          <stddev>0.005</stddev>
         </noise>
       </ray>
