Commit message: improved nav2 params

File: src/wd_lift_robot/urdf/robot.urdf.xacro (robot description, xacro)
@@ -166,6 +166,6 @@
     <origin xyz="0 0 0.25" rpy="0 0 0"/>
   </joint>
-  <!-- LiDAR Sensor - IMPROVED RANGE -->
-  <link name="laser">
+  <!-- LiDAR Sensor - Fixed frame name consistency -->
+  <link name="lidar_link">
     <visual>
       <origin xyz="0 0 0" rpy="0 0 0"/>
@@ -187,7 +187,7 @@
     </inertial>
   </link>
-  <joint name="laser_joint" type="fixed">
+  <joint name="lidar_joint" type="fixed">
     <parent link="base_link"/>
-    <child link="laser"/>
+    <child link="lidar_link"/>
     <origin xyz="0.15 0 ${base_height/2 + 0.02}" rpy="0 0 0"/>
   </joint>
@@ -200,6 +200,6 @@
     <joint name="front_left_wheel_joint">
       <command_interface name="velocity">
-        <param name="min">-50</param>
-        <param name="max">50</param>
+        <param name="min">-10</param>
+        <param name="max">10</param>
       </command_interface>
       <state_interface name="velocity"/>
@@ -208,6 +208,6 @@
     <joint name="front_right_wheel_joint">
       <command_interface name="velocity">
-        <param name="min">-50</param>
-        <param name="max">50</param>
+        <param name="min">-10</param>
+        <param name="max">10</param>
       </command_interface>
       <state_interface name="velocity"/>
@@ -216,6 +216,6 @@
     <joint name="rear_left_wheel_joint">
       <command_interface name="velocity">
-        <param name="min">-50</param>
-        <param name="max">50</param>
+        <param name="min">-10</param>
+        <param name="max">10</param>
       </command_interface>
       <state_interface name="velocity"/>
@@ -224,6 +224,6 @@
     <joint name="rear_right_wheel_joint">
       <command_interface name="velocity">
-        <param name="min">-50</param>
-        <param name="max">50</param>
+        <param name="min">-10</param>
+        <param name="max">10</param>
       </command_interface>
       <state_interface name="velocity"/>
@@ -234,5 +234,5 @@
       <command_interface name="position">
         <param name="min">0</param>
-        <param name="max">0.8</param>
+        <param name="max">0.5</param>
       </command_interface>
       <state_interface name="position"/>
@@ -250,5 +250,5 @@
     <material>Gazebo/Blue</material>
   </gazebo>
-  <!-- Wheel physics -->
+  <!-- Wheel physics with correct friction -->
   <gazebo reference="front_left_wheel">
     <material>Gazebo/Black</material>
@@ -291,15 +291,15 @@
     <fdir1>1 0 0</fdir1>
   </gazebo>
-  <!-- LiDAR sensor plugin - IMPROVED -->
-  <gazebo reference="laser">
+  <!-- LiDAR sensor plugin with correct frame name -->
+  <gazebo reference="lidar_link">
     <material>Gazebo/Black</material>
     <sensor type="ray" name="rplidar_a1">
       <pose>0 0 0 0 0 0</pose>
-      <visualize>false</visualize>  <!-- Reduced visualization load -->
-      <update_rate>20</update_rate>  <!-- Reduced from 30 to 20 Hz -->
+      <visualize>true</visualize>
+      <update_rate>15</update_rate>
       <ray>
         <scan>
           <horizontal>
-            <samples>360</samples>  <!-- Reduced from 720 to 360 -->
+            <samples>360</samples>
             <resolution>1</resolution>
             <min_angle>-3.14159265</min_angle>
@@ -308,12 +308,12 @@
         </scan>
         <range>
-          <min>0.12</min>  <!-- Slightly increased min range -->
-          <max>8.0</max>   <!-- Reduced from 15.0 to 8.0 for indoor use -->
-          <resolution>0.02</resolution>  <!-- Slightly increased resolution -->
+          <min>0.15</min>
+          <max>12.0</max>
+          <resolution>0.01</resolution>
         </range>
         <noise>
           <type>gaussian</type>
           <mean>0.0</mean>
-          <stddev>0.01</stddev>  <!-- Slightly increased noise for realism -->
+          <stddev>0.01</stddev>
         </noise>
       </ray>
@@ -324,5 +324,5 @@
         </ros>
         <output_type>sensor_msgs/LaserScan</output_type>
-        <frame_name>laser</frame_name>
+        <frame_name>lidar_link</frame_name>
       </plugin>
     </sensor>
